File: Power Board/EEE3088F Power Board/EEE3088F Power Board.kicad_sch (KiCad schematic)
At the start: 67 parts, among them J1 Conn_02x16_Odd_Even, J2 USB_C_Receptacle, Q1 2N7002, U1 INA219AxDCN, U2 LM2596S-5, U3 TP4056-42-ESOP8, U4 DRV8837, U5 DRV8837, U6 DRV8837, U7 DRV8837, U8 TPS63020DSJR, U9 CH224K

Commit message: Basic schematic finished
Parts:
- removed JP1: SolderJumper_2_Open, symbol Jumper:SolderJumper_2_Open
- added C15, C25: 1u, Capacitor_SMD:C_0402_1005Metric_Pad0.74x0.62mm_HandSolder, symbol Device:C_Small
- added C16: 1n, symbol Device:C_Small
- added C17: 1n, Capacitor_SMD:C_0603_1608Metric_Pad1.08x0.95mm_HandSolder, symbol Device:C_Small
- added C18, C19: 10u, symbol Device:C
- added C20: 100n, symbol Device:C
- added C21, C22, C23, C24: 22u, symbol Device:C
- added D5: LED, symbol Device:LED
- added J3: Conn_01x02_Socket, Connector_JST:JST_PH_S2B-PH-K_1x02_P2.00mm_Horizontal, symbol Connector:Conn_01x02_Socket
- added L3: 1.5uH, symbol Device:L
- added Rfb3, Rpg2: 1M, symbol Device:R_US
- added Rfb4: 120k, symbol Device:R_US
- added SW1: SW_SPDT_312, symbol Switch:SW_SPDT_312
- added TP18, TP19, TP20, TP21, TP26, TP27: TestPoint, TestPoint:TestPoint_Pad_D2.0mm, symbol Connector:TestPoint
- added TP22: 5V_out, symbol Connector:TestPoint
- added TP23: Ind_chng, symbol Connector:TestPoint
- added TP24: Bias1, symbol Connector:TestPoint
- added TP25: TestPoint, symbol Connector:TestPoint
- added U10: AP22966DC8-7, AP22966DC8-7:IC_AP22966DC8-7, symbol AP22966DC8-7:AP22966DC8-7
- added U11: TPS63020DSJR, TPS63020DSJR:IC_TPS63020DSJR, symbol TPS63020DSJR:TPS63020DSJR
- Rfb1: value 1.232M -> 1.M
- Rfb2: value 220k -> 180k
- renumbered R to R11
Connections:
- net +Batt: now also SW1.2 (C)
- net CTRL_EXT_LOAD1: now also U10.3 (EN1)
- net CTRL_EXT_LOAD2: now also U10.5 (EN2)
- net EXT_LOAD1_OUT: now also TP19.1, U10.13_14 (VOUT1)
- net EXT_LOAD2_OUT: now also TP18.1, U10.8_9 (VOUT2)
- net GND: now also C15.2, C16.1, C17.1, C18.1, C19.1, C20.1, C21.1, C22.1, C23.1, C24.1, C25.2, D5.1 (K), Rfb4.2, SW1.3 (A), U10.11 (GND), U11.15 (PGND), U11.2 (GND)
- net Switch-: now also C12.2, C6.2, U8.10 (VIN_10), U8.11 (VIN_11), C18.2, C19.2, SW1.1 (B), U11.10 (VIN_10), U11.11 (VIN_11)
- new net: J3.1 (Pin_1), TP27.1
- new net: Rfb3.2, Rfb4.1, TP24.1, U11.3 (FB)
- new net: C17.2, U10.10 (SS2)
- new net: C20.2, U11.1 (VINA), U11.12 (EN), U11.13 (PS/SYNC)
- new net: D5.2 (A), Rpg2.2, U11.14 (PG)
- new net: L3.2, TP23.1, U11.6 (L2_6), U11.7 (L2_7)
- new net: L3.1, TP25.1, U11.8 (L1_8), U11.9 (L1_9)
- new net: C16.2, U10.12 (SS1)
- new net: J3.2 (Pin_2), TP26.1
- new net +3V3: TP21.1, U10.4 (VBIAS)
- new net +5V: C15.1, C21.2, C22.2, C23.2, C24.2, C25.1, Rfb3.1, Rpg2.1, TP20.1, TP22.1, U10.1_2 (VIN1), U10.6_7 (VIN2), U11.4 (VOUT_4), U11.5 (VOUT_5)
Other:
- note added: "- 99% Sure correct FP (same dim) - Check orientation (which wire +- fits in which side) - Test points to bypass if incorrect - Do not pupulate (Given)"
- note added: "- Defualt SW_SPDT symbol - Pulls power from circuit"
- note added: "- Double check the Cap values - What is EXP? Base plate contact maybe - Check this is 100% the right symbol. The other pins are correct, just concerend abt 15 - I think this is the packafe with exposed PAD for thermal - base - Add LED indicator?"
- note added: "-Add in the 5V (same circuit with diff FB) when footprints are complete - Check what pwr req from L and if can be basic - Rename components - Check if LED correct from PG - Is EN not meant to be high? - Add / Fix Jumers and TPs - Footprint for passives - Might need to adjust resistor values to ensure basic"
- note added: "Battery Pins"
- note added: "Manual Switch"
- note added: "Power Regulation"
- note added: "Soft Start Caps (up to 25V)"
- note added: "To Do list in a suggestive order: 1) Clarity on our design assumptions 2) Check all design logic (esp Volt reg values), check eachothers Add testing procedure comments and test points. 3) Assign footprints (check with eachother as we go. This is the biggest killer of PCBs. This includes passives and ensuring basic passives available on JLC Have chats with others abt plugin and finding footprints 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"
- note removed: "-Add in the 5V (same circuit with diff FB) when footprints are complete - Check what pwr req from L and if can be basic - Rename components - Check if LED correct from PG - Is EN not meant to be high? - Add / Fix Jumers and TPs - Footprint for passives"
- note removed: "Power Regulation & Swtich"
- moved on the sheet: U4, U5, U6, U7

Commit message: annotations, test points
Parts:
- added JP1: SolderJumper_2_Open, symbol Jumper:SolderJumper_2_Open
Connections:
- net V_bus is gone; now on net HV: J2.A4 (VBUS), J2.A9 (VBUS), J2.B4 (VBUS), J2.B9 (VBUS), R10.1, R9.1, TP6.1
- net +Batt: no longer C5.1, TP15.1, U3.5 (BAT), U4.1 (VM), U5.1 (VM), U6.1 (VM), U7.1 (VM)
- net Battery: now also C5.1, TP15.1, U3.5 (BAT), U4.1 (VM), U5.1 (VM), U6.1 (VM), U7.1 (VM); no longer C2.1, U2.1 (VIN)
- net HV: now also C2.1, U2.1 (VIN)
Other:
- note added: "+D and -D tracks must be same length!!"
- note added: "add P MOSFET between Vbus and HV?"
- note added: "if transistor config around fast charge control doesn't work, disconnect transistor @jumper to have only slow charging mode"
- moved on the sheet: R4, TP12, TP15

Commit message: checked FP PWR reg and Curr Sens
Parts:
- removed C10, C11, C21, C23, C24, C8, C9: 22u, symbol Device:C
- removed C12, C18, C6: 10u, symbol Device:C
- removed C20, C7: 100n, symbol Device:C
- removed D4: LED, symbol Device:LED
- removed JP2: Jumper_2_Bridged, TestPoint:TestPoint_Pad_D2.0mm, symbol Jumper:Jumper_2_Bridged
- removed L2: 1.5uH, symbol Device:L
- removed Rfb1: 1.M, symbol Device:R_US
- removed Rfb2: 180k, symbol Device:R_US
- removed Rfb3, Rpg1: 1M, symbol Device:R_US
- removed Rfb4: 120k, symbol Device:R_US
- removed TP1, TP24: Bias1, symbol Connector:TestPoint
- removed TP2: 3v3_out, symbol Connector:TestPoint
- removed TP22: 5V_out, symbol Connector:TestPoint
- removed TP23, TP3: Ind_chng, symbol Connector:TestPoint
- removed TP25, TP4: TestPoint, symbol Connector:TestPoint
- removed U11, U8: TPS63020DSJR, TPS63020DSJR:IC_TPS63020DSJR, symbol TPS63020DSJR:TPS63020DSJR
- added C_P(in)1: 10u, Capacitor_SMD:C_0603_1608Metric_Pad1.08x0.95mm_HandSolder, symbol Device:C
- added C_P(in)2, C_P(out)2, C_P(out)3: 22u, Capacitor_SMD:C_0603_1608Metric_Pad1.08x0.95mm_HandSolder, symbol Device:C
- added D6: LED_P2, LED_SMD:LED_0805_2012Metric_Pad1.15x1.40mm_HandSolder, symbol Device:LED
- added JPI1: I2C_PU, Jumper:SolderJumper-2_P1.3mm_Open_RoundedPad1.0x1.5mm, symbol Jumper:SolderJumper_2_Open
- added JPI2: 219_PWR, Jumper:SolderJumper-2_P1.3mm_Open_RoundedPad1.0x1.5mm, symbol Jumper:SolderJumper_2_Open
- added JPI3: SHUNT, Jumper:SolderJumper-2_P1.3mm_Open_RoundedPad1.0x1.5mm, symbol Jumper:SolderJumper_2_Open
- added JP_P1: Boost_PWR, Jumper:SolderJumper-2_P1.3mm_Open_RoundedPad1.0x1.5mm, symbol Jumper:SolderJumper_2_Open
- added JP_P2: Boost_MODE, Jumper:SolderJumper-2_P1.3mm_Open_RoundedPad1.0x1.5mm, symbol Jumper:SolderJumper_2_Open
- added R_P2: 1k, Resistor_SMD:R_0603_1608Metric_Pad0.98x0.95mm_HandSolder, symbol Device:R_US
- added R_Pfb1: 732k, Resistor_SMD:R_0603_1608Metric_Pad0.98x0.95mm_HandSolder, symbol Device:R_US
- added R_Pfb2: 100k, Resistor_SMD:R_0603_1608Metric_Pad0.98x0.95mm_HandSolder, symbol Device:R_US
- added TP_P1, TP_P2: Boost_ind, TestPoint:TestPoint_Pad_D2.0mm, symbol Connector:TestPoint
- added TP_P3: 5V_OUT, TestPoint:TestPoint_Pad_D2.0mm, symbol Connector:TestPoint
- added TP_P4: Feedback1, TestPoint:TestPoint_Pad_D2.0mm, symbol Connector:TestPoint
- added TP_P5: GND, TestPoint:TestPoint_Pad_D2.0mm, symbol Connector:TestPoint
- added TP_P6: 3V3_OUT, TestPoint:TestPoint_Pad_D2.0mm, symbol Connector:TestPoint
- added U_P1: TPS61022, Package_DFN_QFN:Texas_RWU0007A_VQFN-7_2x2mm_P0.5mm, symbol Converter_DCDC:TPS61022
- added U_P2: AMS1117-3.3, Package_TO_SOT_SMD:SOT-223-3_TabPin2, symbol Regulator_Linear:AMS1117-3.3
- C_I(in): renamed from C1; footprint (none) -> Capacitor_SMD:C_0603_1608Metric_Pad1.08x0.95mm_HandSolder
- C_P(in): renamed from C19; footprint (none) -> Capacitor_SMD:C_0603_1608Metric_Pad1.08x0.95mm_HandSolder
- C_P(out)1: renamed from C22; footprint (none) -> Capacitor_SMD:C_0603_1608Metric_Pad1.08x0.95mm_HandSolder
- D5: value LED -> LED__P1
- L3: value 1.5uH -> 1uH
- R_I1: renamed from Rpullup2; footprint (none) -> Resistor_SMD:R_0603_1608Metric_Pad0.98x0.95mm_HandSolder
- R_I2: renamed from Rpullup1; footprint (none) -> Resistor_SMD:R_0603_1608Metric_Pad0.98x0.95mm_HandSolder
- R_Ishunt: renamed from Shunt_res1; footprint (none) -> Resistor_SMD:R_1206_3216Metric_Pad1.30x1.75mm_HandSolder
- R_P1: renamed from Rpg2; value 1M -> 1k; footprint (none) -> Resistor_SMD:R_0603_1608Metric_Pad0.98x0.95mm_HandSolder
- U1: value INA219AxDCN -> INA219AIDCNR
- renumbered TP27 to Batt+, TP26 to Batt-
Connections:
- net +Batt is gone; now on net Battery: SW1.2 (C)
- net 3V3 Out is gone; now on net +3V3: J1.18 (Pin_18), U4.7 (~{SLEEP}), U4.8 (VCC), U5.7 (~{SLEEP}), U5.8 (VCC), U6.7 (~{SLEEP}), U6.8 (VCC), U7.7 (~{SLEEP}), U7.8 (VCC)
- net Battery_Side is gone; now on net Batt+: R_Ishunt.2, U1.2 (IN-)
- net Charger_Side_ is gone; now on net Battery: R_Ishunt.1, U1.1 (IN+)
- net +3.3V: now also JPI1.1 (A), JPI2.1 (A); no longer C_I(in).2, U1.4 (VS)
- net +3V3: now also C_P(in)2.2, R_P2.1, TP_P6.1, U_P2.2 (VO)
- net +5V: now also C_P(in)1.2, C_P(out)2.2, C_P(out)3.2, R_Pfb1.1, TP_P3.1, U_P1.3 (VOUT), U_P2.3 (VI)
- net Battery: now also JPI3.2 (B), JP_P1.2 (B)
- net GND: now also C_P(in)1.1, C_P(in)2.1, C_P(out)2.1, C_P(out)3.1, D6.1 (K), R_Pfb2.2, TP_P5.1, U_P1.1 (GND), U_P2.1 (GND)
- net Switch-: no longer C_P(in).2
- net Batt+: now reaches Batt+.1, J3.1 (Pin_1)
- net Batt+: now also JPI3.1 (A)
- net at R_I1.1, R_I2.1: now also JPI1.2 (B)
- net at L3.2: now also TP_P2.1, U_P1.2 (SW)
- net at L3.1: now also C_P(in).2, JP_P1.1 (A), JP_P2.2 (B), TP_P1.1, U_P1.5 (EN), U_P1.7 (VIN)
- new net: R_Pfb1.2, R_Pfb2.1, TP_P4.1, U_P1.4 (FB)
- new net: D6.2 (A), R_P2.2
- new net: C_I(in).2, JPI2.2 (B), U1.4 (VS)
- new net: JP_P2.1 (A), U_P1.6 (MODE)
Other:
- note added: "- Check what pwr req from L and if can be basic - Rename components - Check if LED correct from PG - Is EN not meant to be high? - Add / Fix Jumers and TPs - Footprint for passives - Might need to adjust resistor values to ensure basic"
- note added: "2.7V to 4.2V"
- note added: "Boost Converter"
- note added: "Can get away with ceramic"
- note added: "High EN-> Forced PWM for heavy load Design taken from DS Ensure small loop in PCB"
- note added: "INA219AIDCNR Current Sensor - I"
- note added: "LDO 5V->3V3"
- note added: "Load Switching-L"
- note added: "Specific Shunt Res"
- note added: "Vout to Cap < 4cm"
- note added: "must still determine which inductor. REQ: Value = 1u Low Sat current DCR"
- note removed: "-Add in the 5V (same circuit with diff FB) when footprints are complete - Check what pwr req from L and if can be basic - Rename components - Check if LED correct from PG - Is EN not meant to be high? - Add / Fix Jumers and TPs - Footprint for passives - Might need to adjust resistor values to ensure basic"
- note removed: "INA219AIDCNR Current Sensor"
- note removed: "Imported Symbol"
- note removed: "Load Switching"
- moved on the sheet: C_P(in), C_P(out)1, D5, R_P1

Commit message: IC and passive component footprints added
Parts:
- removed R1, R10, R2: 1k, symbol Device:R
- removed R3: 0.4R, symbol Device:R
- removed R4: 2k7, 0805W8F2701T5E, symbol Device:R
- removed R5: 5k6, 0805W8F5601T5E, symbol Device:R
- removed R6: 100R, 1206W4F1000T5E, symbol Device:R
- removed R7, R9: 10k, symbol Device:R
- removed R8: 6k8, symbol Device:R
- removed U7: DRV8837, Package_SON:WSON-8-1EP_2x2mm_P0.5mm_EP0.9x1.6mm, symbol Driver_Motor:DRV8837
- added R12, R13, R22: 1k, Resistor_SMD:R_0603_1608Metric_Pad0.98x0.95mm_HandSolder, symbol Device:R_US
- added R14: 2k7, Resistor_SMD:R_0603_1608Metric_Pad0.98x0.95mm_HandSolder, symbol Device:R_US
- added R15: 5k6, Resistor_SMD:R_0603_1608Metric_Pad0.98x0.95mm_HandSolder, symbol Device:R_US
- added R16: 100R, Resistor_SMD:R_0603_1608Metric_Pad0.98x0.95mm_HandSolder, symbol Device:R_US
- added R17, R23: 10k, Resistor_SMD:R_0603_1608Metric_Pad0.98x0.95mm_HandSolder, symbol Device:R_US
- added R18, R19, R20, R21: 0.1R, Resistor_SMD:R_1206_3216Metric_Pad1.30x1.75mm_HandSolder, symbol Device:R_US
- added R24: 6k8, Resistor_SMD:R_0603_1608Metric_Pad0.98x0.95mm_HandSolder, symbol Device:R_US
- added U8: DRV8837, DRV8837DSGR:SON50P200X200X80-9N, symbol Driver_Motor:DRV8837
- C13, C4, C5: footprint (none) -> Capacitor_SMD:C_0603_1608Metric_Pad1.08x0.95mm_HandSolder
- L1: value 68uH -> 22uH
- U2: value LM2596S-5 -> LM2596SX-5.0/NOPB; footprint Package_TO_SOT_SMD:TO-263-5_TabPin3 -> LM2596SX-5.0_NOPB:VREG_LM2596SX-5.0_NOPB
- U3: footprint Package_SO:SOIC-8-1EP_3.9x4.9mm_P1.27mm_EP2.41x3.3mm_ThermalVias -> TP4056-42-ESOP8:SOIC127P600X175-9N
- U4, U5, U6: footprint Package_SON:WSON-8-1EP_2x2mm_P0.5mm_EP0.9x1.6mm -> DRV8837DSGR:SON50P200X200X80-9N
Connections:
- net +3V3: now also U8.7 (~{SLEEP}), U8.8 (VCC)
- net 5V_Buck_Out: now also R21.1
- net Battery: now also U8.1 (VM)
- net FAST_CHARGE_CTRL: now also R16.1
- net GND: now also R15.2, R17.2, R24.2, U8.4 (GND), U8.9 (GND)
- net HV: now also R22.1, R23.1
- net MOTOR1_CTRL1: now also U8.6 (IN1); no longer U6.6 (IN1)
- net MOTOR1_CTRL2: now also U8.5 (IN2); no longer U6.5 (IN2)
- net MOTOR3_CTRL1: now also U6.6 (IN1)
- net MOTOR3_CTRL2: now also U6.5 (IN2)
- net Motor1_A_OUT: now also U8.2 (OUT1); no longer U6.2 (OUT1)
- net Motor1_B_OUT: now also U8.3 (OUT2); no longer U6.3 (OUT2)
- net Motor3_A_OUT: now also U6.2 (OUT1)
- net Motor3_B_OUT: now also U6.3 (OUT2)
- net at TP10.1, U3.2 (PROG): now also R14.1, R15.1
- net at C4.1, D2.2 (A), D3.2 (A)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: now also R18.2
- net at U3.6 (~{STDBY}): now also R13.2
- net at U3.7 (~{CHRG}): now also R12.2
- net at C13.1, TP7.1, U9.1 (VDD): now also R22.2
- net at Q1.1 (G), TP13.1: now also R16.2, R17.1
- net at Q1.3 (D), TP12.1: now also R14.2
- net at D3.1 (K): now also R12.1
- net at U9.8 (VBUS): now also R23.2
- net at TP9.1, U9.9 (CFG1): now also R24.1
- net at D2.1 (K): now also R13.1
- new net: R19.1, R20.2
- new net: R18.1, R19.2
- new net: R20.1, R21.2
Other:
- note added: "- add jumpers and test points - check capacitor/inductor values - decide on LED components & colours - find components for in and out caps - LED footprints"
- note added: "Can't find basic 0.4R resistor, can only find basic 0.1R"
- note added: "Do capacitor and inductor values need to be exact? Save budget"
- note added: "Done: - Resistors and Capacitors footprints (except LM256) - IC footprints - Schottky diode and 2N7002 footprints To Do: - LED footprints - LM256 caps and inductor? - ask about 0.4R resistor - Neaten net labels - relabel passive components"
- note removed: "- add jumpers and test points - check capacitor/inductor values - check that MOSFET doesnt disrupt Rprog reading - decide on LED components & colours"
