File: Power Board/EEE3088F Power Board/EEE3088F Power Board.kicad_sch (KiCad schematic)
At the start: 92 parts, among them J1 Conn_02x16_Odd_Even, J2 USB_C_Receptacle, J3 Conn_01x02_Socket, Q1 2N7002, U1 INA219AIDCNR, U10 DRV8837DSGR, U11 DRV8837DSGR, U12 DRV8837DSGR, U13 DRV8837DSGR, U2 TPS5430DDA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

Commit message: killing the mac version
Parts:
- added JP_B1: charge_in, Jumper:SolderJumper-2_P1.3mm_Open_RoundedPad1.0x1.5mm, symbol Jumper:SolderJumper_2_Open
- added JP_B2: buck_charge, Jumper:SolderJumper-2_P1.3mm_Open_RoundedPad1.0x1.5mm, symbol Jumper:SolderJumper_2_Open
- added JP_Bout: charge_batt+, Jumper:SolderJumper-2_P1.3mm_Open_RoundedPad1.0x1.5mm, symbol Jumper:SolderJumper_2_Open
- added JP_Bprog: fast_prog, Jumper:SolderJumper-2_P1.3mm_Open_RoundedPad1.0x1.5mm, symbol Jumper:SolderJumper_2_Open
- added JP_C1: vbus, Jumper:SolderJumper-2_P1.3mm_Open_RoundedPad1.0x1.5mm, symbol Jumper:SolderJumper_2_Open
- added TP_P7: TP_VM, TestPoint:TestPoint_Pad_D2.0mm, symbol Connector:TestPoint
- TP10: value TestPoint -> charge_prog
- TP11: value TestPoint -> charge_gnd
Connections:
- net -BATT is gone; now on net GND: Batt-1.1, J3.2 (Pin_2)
- net +9V: now also JP_B1.2 (B), JP_C1.2 (B); no longer C_Bin1.1, J2.A4 (VBUS), J2.A9 (VBUS), J2.B4 (VBUS), J2.B9 (VBUS), U2.7 (VIN)
- net +BATT: now also J1.14 (Pin_14), JPI3.2 (B), R_Ishunt1.1, SW1.1, U1.1 (IN+)
- net 5V_Buck_Out: now also JP_B2.1 (A); no longer C_B3.1, L1.2, R_Bset1.1
- net Batt+: now also TP15.1, U10.1 (VM), U11.1 (VM), U12.1 (VM), U13.1 (VM), JP_Bout.2 (B), TP_P7.1
- net at R_B_slow1.1, TP10.1, U3.2 (PROG): now also JP_Bprog.1 (A); no longer R_B_fast1.1
- removed net Battery: C_B2.1, J1.14 (Pin_14), JPI3.2 (B), R_Ishunt1.1, SW1.1, TP15.1, U1.1 (IN+), U10.1 (VM), U11.1 (VM), U12.1 (VM), U13.1 (VM), U3.5 (BAT)
- new net: J2.A4 (VBUS), J2.A9 (VBUS), J2.B4 (VBUS), J2.B9 (VBUS), JP_C1.1 (A)
- new net: C_B2.1, JP_Bout.1 (A), U3.5 (BAT)
- new net: JP_Bprog.2 (B), R_B_fast1.1
- new net: C_B3.1, JP_B2.2 (B), L1.2, R_Bset1.1
- new net: C_Bin1.1, JP_B1.1 (A), U2.7 (VIN)
Other:
- note removed: "jump"
- moved on the sheet: R_B_fast1

Commit message: finished schematic
Other:
- note removed: "**fix footprint"
- note removed: "- add jumpers and test points - check capacitor/inductor values - decide on LED components & colours - find components for in and out caps - LED footprints"
- note removed: "Cap V rating > 1.5xVout"
- note removed: "Do capacitor and inductor values need to be exact? Save budget If so, is it worth changing my whole design to find a different buck convertor that doesn't use extended caps"
- note removed: "add P MOSFET between Vbus and HV?"
- note removed: "found a 22uH extended preferred but stock count 307??"
- note removed: "jump 3V3 Out jump +Batt"
- note removed: "jump each IC?"
- moved on the sheet: C_B3, C_Bboot1, C_Bin1, D4, JP_B1, JP_B2, JP_M_3V3, L1, R_Bset1, R_Bset2, TP17, U2
