File: Power Board/EEE3088F Power Board/NEW_KICAD/Power_Board_3088F.kicad_pcb (KiCad board)
At the start: 2 copper layers, 92 parts, among them J1 Conn_02x16_Odd_Even, J2 USB_C_Receptacle, J3 Conn_01x02_Socket, Q1 2N7002, U1 INA219AIDCNR, U10 DRV8837DSGR, U11 DRV8837DSGR, U12 DRV8837DSGR, U13 DRV8837DSGR, U2 TPS5430DDA, U3 TP4056-42-ESOP8, U7 AP22966DC8-7, U9 CH224K

Commit message: finished schematic
Parts:
- removed Batt+1, Batt-1, TP10, TP11, TP12, TP13, TP14, TP15, TP17, TP18, TP19, TP21, TP6, TP7, TP8, TP9: TestPoint, TestPoint:TestPoint_Pad_D2.0mm
- removed C15, C25: 1u, Capacitor_SMD:C_0603_1608Metric_Pad1.08x0.95mm_HandSolder
- removed C16, C17: 1n, Capacitor_SMD:C_0603_1608Metric_Pad1.08x0.95mm_HandSolder
- removed C_B1, C_B2: 10uF, Capacitor_SMD:C_0603_1608Metric_Pad1.08x0.95mm_HandSolder
- removed C_B3: 220uF, Capacitor_SMD:CP_Elec_6.3x7.7
- removed C_Bboot1: 10nF, Capacitor_SMD:C_0603_1608Metric_Pad1.08x0.95mm_HandSolder
- removed C_Bin1: 10uF, Capacitor_SMD:C_1206_3216Metric_Pad1.33x1.80mm_HandSolder
- removed C_C_dd1: 1uF, Capacitor_SMD:C_0603_1608Metric_Pad1.08x0.95mm_HandSolder
- removed C_I(in)1: 100n, Capacitor_SMD:C_0603_1608Metric_Pad1.08x0.95mm_HandSolder
- removed C_P(in)1, C_P(in)3: 10u, Capacitor_SMD:C_0603_1608Metric_Pad1.08x0.95mm_HandSolder
- removed C_P(in)2, C_P(out)1, C_P(out)2, C_P(out)3: 22u, Capacitor_SMD:C_0603_1608Metric_Pad1.08x0.95mm_HandSolder
- removed D2: Red LED, LED_SMD:LED_0603_1608Metric_Pad1.05x0.95mm_HandSolder
- removed D3: Green LED, LED_SMD:LED_0805_2012Metric_Pad1.15x1.40mm_HandSolder
- removed D4: BA340A, custom_footprints:SMA-DIODE
- removed D5: LED__P1, LED_SMD:LED_0805_2012Metric_Pad1.15x1.40mm_HandSolder
- removed D6: LED_P2, LED_SMD:LED_0805_2012Metric_Pad1.15x1.40mm_HandSolder
- removed J1: Conn_02x16_Odd_Even, Connector_PinHeader_2.54mm:PinHeader_2x16_P2.54mm_Vertical
- removed J2: USB_C_Receptacle, Connector_USB:USB_C_Receptacle_G-Switch_GT-USB-7010ASV
- removed J3: Conn_01x02_Socket, Connector_JST:JST_PH_S2B-PH-K_1x02_P2.00mm_Horizontal
- removed JPI1: I2C_PU, Jumper:SolderJumper-2_P1.3mm_Open_RoundedPad1.0x1.5mm
- removed JPI2: 219_PWR, Jumper:SolderJumper-2_P1.3mm_Open_RoundedPad1.0x1.5mm
- removed JPI3: SHUNT, Jumper:SolderJumper-2_P1.3mm_Open_RoundedPad1.0x1.5mm
- removed JPI4: VIN1, Jumper:SolderJumper-2_P1.3mm_Open_RoundedPad1.0x1.5mm
- removed JPI5: VIN2, Jumper:SolderJumper-2_P1.3mm_Open_RoundedPad1.0x1.5mm
- removed JPI6: VBIAS, Jumper:SolderJumper-2_P1.3mm_Open_RoundedPad1.0x1.5mm
- removed JP_M_3V3: 3V3_VM, Jumper:SolderJumper-2_P1.3mm_Open_RoundedPad1.0x1.5mm
- removed JP_P1: Boost_PWR, Jumper:SolderJumper-2_P1.3mm_Open_RoundedPad1.0x1.5mm
- removed JP_P2: Boost_MODE, Jumper:SolderJumper-2_P1.3mm_Open_RoundedPad1.0x1.5mm
- removed JP_P3: LDO_PWR, Jumper:SolderJumper-2_P1.3mm_Open_RoundedPad1.0x1.5mm
- removed L1: 18uH, Inductor_SMD:L_Abracon_ASPI-4030S
- removed L3: 1uH, Inductor_SMD:L_Changjiang_FXL0630
- removed Q1: 2N7002, Package_TO_SOT_SMD:SOT-23
- removed R19, R20: 1R, Resistor_SMD:R_0603_1608Metric_Pad0.98x0.95mm_HandSolder
- removed R_B_LED1, R_B_LED2, R_C_dd1, R_P1, R_P2: 1k, Resistor_SMD:R_0603_1608Metric_Pad0.98x0.95mm_HandSolder
- removed R_B_b1: 100R, Resistor_SMD:R_0603_1608Metric_Pad0.98x0.95mm_HandSolder
- removed R_B_fast1: 2k7, Resistor_SMD:R_0603_1608Metric_Pad0.98x0.95mm_HandSolder
- removed R_B_pd1, R_Bset1, R_C_bus1: 10k, Resistor_SMD:R_0603_1608Metric_Pad0.98x0.95mm_HandSolder
- removed R_B_slow1: 5k6, Resistor_SMD:R_0603_1608Metric_Pad0.98x0.95mm_HandSolder
- removed R_Bset2: 3k3, Resistor_SMD:R_0603_1608Metric_Pad0.98x0.95mm_HandSolder
- removed R_C_cfg1: 6k8, Resistor_SMD:R_0603_1608Metric_Pad0.98x0.95mm_HandSolder
- removed R_I1, R_I2: 3.3k, Resistor_SMD:R_0603_1608Metric_Pad0.98x0.95mm_HandSolder
- removed R_Ishunt1: 0.1, Resistor_SMD:R_1206_3216Metric_Pad1.30x1.75mm_HandSolder
- removed R_Pfb1: 510k, Resistor_SMD:R_0603_1608Metric_Pad0.98x0.95mm_HandSolder
- removed R_Pfb2: 68k, Resistor_SMD:R_0603_1608Metric_Pad0.98x0.95mm_HandSolder
- removed SW1: ~, custom_footprints:SW-TH_SS-12D11G5
- removed TP_P1, TP_P2: Boost_ind, TestPoint:TestPoint_Pad_D2.0mm
- removed TP_P3: 5V_OUT, TestPoint:TestPoint_Pad_D2.0mm
- removed TP_P4: Feedback1, TestPoint:TestPoint_Pad_D2.0mm
- removed TP_P5: GND, TestPoint:TestPoint_Pad_D2.0mm
- removed TP_P6: 3V3_OUT, TestPoint:TestPoint_Pad_D2.0mm
- removed U1: INA219AIDCNR, Package_TO_SOT_SMD:SOT-23-8
- removed U10, U11, U12, U13: DRV8837DSGR, custom_footprints:SON50P200X200X80-9N
- removed U2: TPS5430DDA, Package_SO:SOIC-8-1EP_3.9x4.9mm_P1.27mm_EP2.29x3mm
- removed U3: TP4056-42-ESOP8, custom_footprints:SOIC127P600X175-9N
- removed U7: AP22966DC8-7, custom_footprints:IC_AP22966DC8-7
- removed U9: CH224K, Package_SO:SSOP-10-1EP_3.9x4.9mm_P1mm_EP2.1x3.3mm
- removed U_P1: TPS61022, Package_DFN_QFN:Texas_RWU0007A_VQFN-7_2x2mm_P0.5mm
- removed U_P2: AMS1117-3.3, Package_TO_SOT_SMD:SOT-223-3_TabPin2

Commit message: pcb islands done
Parts:
- added 3V3: LED_P2, LED_SMD:LED_0603_1608Metric_Pad1.05x0.95mm_HandSolder, F.Cu at (198.0, 158.0)
- added 5V0: LED__P1, LED_SMD:LED_0603_1608Metric_Pad1.05x0.95mm_HandSolder, F.Cu at (155.3, 171.0)
- added Batt+1: TestPoint, TestPoint:TestPoint_Pad_D2.0mm, F.Cu at (100.0, 92.0)
- added Batt-1: TestPoint, TestPoint:TestPoint_Pad_D2.0mm, F.Cu at (93.2, 94.7)
- added C15: 1u, Capacitor_SMD:C_0603_1608Metric_Pad1.08x0.95mm_HandSolder, F.Cu at (37.6, 29.0)
- added C16: 1n, Capacitor_SMD:C_0603_1608Metric_Pad1.08x0.95mm_HandSolder, F.Cu at (33.9, 31.0)
- added C17: 1n, Capacitor_SMD:C_0603_1608Metric_Pad1.08x0.95mm_HandSolder, F.Cu at (30.6, 33.0)
- added C25: 1u, Capacitor_SMD:C_0603_1608Metric_Pad1.08x0.95mm_HandSolder, F.Cu at (34.7, 35.0)
- added C_B3: 10uF, Capacitor_SMD:C_0603_1608Metric_Pad1.08x0.95mm_HandSolder, F.Cu at (260.9, 94.0)
- added C_B4: 220uF, Capacitor_SMD:CP_Elec_6.3x7.7, F.Cu at (258.0, 159.0)
- added C_B5: 10uF, Capacitor_SMD:C_0603_1608Metric_Pad1.08x0.95mm_HandSolder, F.Cu at (255.5, 96.0)
- added C_Bboot2: 10nF, Capacitor_SMD:C_0603_1608Metric_Pad1.08x0.95mm_HandSolder, F.Cu at (262.9, 151.0)
- added C_Bin2: 10uF, Capacitor_SMD:C_1206_3216Metric_Pad1.33x1.80mm_HandSolder, F.Cu at (278.0, 162.0)
- added C_C_dd1: 1uF, Capacitor_SMD:C_0603_1608Metric_Pad1.08x0.95mm_HandSolder, F.Cu at (48.6, 163.2)
- added C_I(in)1: 100n, Capacitor_SMD:C_0603_1608Metric_Pad1.08x0.95mm_HandSolder, F.Cu at (38.0, 98.0)
- added C_P(in)1: 10u, Capacitor_SMD:C_0603_1608Metric_Pad1.08x0.95mm_HandSolder, F.Cu at (194.9, 147.0)
- added C_P(in)2: 22u, Capacitor_SMD:C_0603_1608Metric_Pad1.08x0.95mm_HandSolder, F.Cu at (187.9, 147.0)
- added C_P(in)3: 10u, Capacitor_SMD:C_0603_1608Metric_Pad1.08x0.95mm_HandSolder, F.Cu at (154.0, 179.0)
- added C_P(out)1: 22u, Capacitor_SMD:C_0603_1608Metric_Pad1.08x0.95mm_HandSolder, F.Cu at (154.9, 184.0)
- added C_P(out)2: 22u, Capacitor_SMD:C_0603_1608Metric_Pad1.08x0.95mm_HandSolder, F.Cu at (163.0, 184.0)
- added C_P(out)3: 22u, Capacitor_SMD:C_0603_1608Metric_Pad1.08x0.95mm_HandSolder, F.Cu at (163.0, 179.0)
- added D4: Red LED, LED_SMD:LED_0603_1608Metric_Pad1.05x0.95mm_HandSolder, F.Cu at (248.7, 58.4)
- added D7: BA340A, custom_footprints:SMA-DIODE, F.Cu at (262.0, 145.0)
- added D8: Green LED, LED_SMD:LED_0603_1608Metric_Pad1.05x0.95mm_HandSolder, F.Cu at (257.0, 59.0)
- added J1: Conn_02x16_Odd_Even, Connector_PinHeader_2.54mm:PinHeader_2x16_P2.54mm_Vertical, F.Cu at (101.6, 30.5)
- added J3: Conn_01x02_Socket, Connector_JST:JST_PH_S2B-PH-K_1x02_P2.00mm_Horizontal, F.Cu at (97.0, 85.5)
- added JPI_3: SHUNT, Jumper:SolderJumper-2_P1.3mm_Open_RoundedPad1.0x1.5mm, F.Cu at (25.3, 106.0)
- added JP_B1: charge_in, Jumper:SolderJumper-2_P1.3mm_Open_RoundedPad1.0x1.5mm, F.Cu at (279.6, 147.0)
- added JP_B2: buck_charge, Jumper:SolderJumper-2_P1.3mm_Open_RoundedPad1.0x1.5mm, F.Cu at (279.9, 140.0)
- added JP_BBatt1: charge_batt+, Jumper:SolderJumper-2_P1.3mm_Open_RoundedPad1.0x1.5mm, F.Cu at (277.6, 74.0)
- added JP_B_ena1: Jumper (leave open), Jumper:SolderJumper-2_P1.3mm_Open_RoundedPad1.0x1.5mm, F.Cu at (276.6, 80.0)
- added JP_Bprog1: fast_prog, Jumper:SolderJumper-2_P1.3mm_Open_RoundedPad1.0x1.5mm, F.Cu at (278.6, 87.0)
- added JP_CVbus1: VBUS, Jumper:SolderJumper-2_P1.3mm_Open_RoundedPad1.0x1.5mm, F.Cu at (55.3, 158.2)
- added JP_I1: 219_PWR, Jumper:SolderJumper-2_P1.3mm_Open_RoundedPad1.0x1.5mm, F.Cu at (31.6, 106.0)
- added JP_I2: I2C_PU, Jumper:SolderJumper-2_P1.3mm_Open_RoundedPad1.0x1.5mm, F.Cu at (39.0, 106.0)
- added JP_L1: VBIAS, Jumper:SolderJumper-2_P1.3mm_Open_RoundedPad1.0x1.5mm, F.Cu at (23.4, 30.0)
- added JP_L2: VIN1, Jumper:SolderJumper-2_P1.3mm_Open_RoundedPad1.0x1.5mm, F.Cu at (23.4, 42.0)
- added JP_L3: VIN2, Jumper:SolderJumper-2_P1.3mm_Open_RoundedPad1.0x1.5mm, F.Cu at (22.4, 36.0)
- added JP_M_3V3: 3V3_VM, Jumper:SolderJumper-2_P1.3mm_Open_RoundedPad1.0x1.5mm, F.Cu at (174.7, 35.2)
- added JP_M_VM1: Batt_VM, Jumper:SolderJumper-2_P1.3mm_Open_RoundedPad1.0x1.5mm, F.Cu at (168.0, 34.2)
- added JP_P1: Boost_ENA, Jumper:SolderJumper-2_P1.3mm_Open_RoundedPad1.0x1.5mm, F.Cu at (145.0, 160.0)
- added JP_P2: Boost_MODE, Jumper:SolderJumper-2_P1.3mm_Open_RoundedPad1.0x1.5mm, F.Cu at (145.0, 166.0)
- added JP_P3: Boost_PWR, Jumper:SolderJumper-2_P1.3mm_Open_RoundedPad1.0x1.5mm, F.Cu at (145.0, 172.0)
- added JP_P4: LDO_PWR, Jumper:SolderJumper-2_P1.3mm_Open_RoundedPad1.0x1.5mm, F.Cu at (188.3, 153.0)
- added L2: 18uH, Inductor_SMD:L_Abracon_ASPI-4030S, F.Cu at (271.0, 145.0)
- added L3: 1uH, Inductor_SMD:L_Changjiang_FXL0630, F.Cu at (138.0, 187.0)
- added Q2: 2N7002, Package_TO_SOT_SMD:SOT-23, F.Cu at (249.9, 68.0)
- added R21: 1R, Resistor_SMD:R_0603_1608Metric_Pad0.98x0.95mm_HandSolder, F.Cu at (266.0, 68.0)
- added R22: 1R, Resistor_SMD:R_0603_1608Metric_Pad0.98x0.95mm_HandSolder, F.Cu at (266.0, 70.5)
- added R_B_LED3: 1k, Resistor_SMD:R_0603_1608Metric_Pad0.98x0.95mm_HandSolder, F.Cu at (258.0, 67.0)
- added R_B_LED4: 1k, Resistor_SMD:R_0603_1608Metric_Pad0.98x0.95mm_HandSolder, F.Cu at (258.0, 72.0)
- added R_B_b2: 100R, Resistor_SMD:R_0603_1608Metric_Pad0.98x0.95mm_HandSolder, F.Cu at (268.0, 77.0)
- added R_B_fast2: 2k7, Resistor_SMD:R_0603_1608Metric_Pad0.98x0.95mm_HandSolder, F.Cu at (261.1, 77.0)
- added R_B_pd2: 10k, Resistor_SMD:R_0603_1608Metric_Pad0.98x0.95mm_HandSolder, F.Cu at (261.1, 82.0)
- added R_B_slow2: 5k6, Resistor_SMD:R_0603_1608Metric_Pad0.98x0.95mm_HandSolder, F.Cu at (260.0, 87.0)
- added R_Bset3: 10k, Resistor_SMD:R_0603_1608Metric_Pad0.98x0.95mm_HandSolder, F.Cu at (250.0, 162.0)
- added R_Bset4: 3k3, Resistor_SMD:R_0603_1608Metric_Pad0.98x0.95mm_HandSolder, F.Cu at (250.0, 157.0)
- added R_C_bus1: 10k, Resistor_SMD:R_0603_1608Metric_Pad0.98x0.95mm_HandSolder, F.Cu at (57.6, 165.1)
- added R_C_cfg1: 6k8, Resistor_SMD:R_0603_1608Metric_Pad0.98x0.95mm_HandSolder, F.Cu at (41.6, 172.2)
- added R_C_dd1: 1k, Resistor_SMD:R_0603_1608Metric_Pad0.98x0.95mm_HandSolder, F.Cu at (42.6, 167.2)
- added R_I1: 3.3k, Resistor_SMD:R_0603_1608Metric_Pad0.98x0.95mm_HandSolder, F.Cu at (38.2, 93.0)
- added R_I2: 3.3k, Resistor_SMD:R_0603_1608Metric_Pad0.98x0.95mm_HandSolder, F.Cu at (42.1, 93.0)
- added R_Ishunt1: 0.1, Resistor_SMD:R_1206_3216Metric_Pad1.30x1.75mm_HandSolder, F.Cu at (25.3, 91.0)
- added R_P1: 1k, Resistor_SMD:R_0603_1608Metric_Pad0.98x0.95mm_HandSolder, F.Cu at (153.0, 165.0)
- added R_P2: 1k, Resistor_SMD:R_0603_1608Metric_Pad0.98x0.95mm_HandSolder, F.Cu at (194.9, 153.0)
- added R_Pfb1: 510k, Resistor_SMD:R_0603_1608Metric_Pad0.98x0.95mm_HandSolder, F.Cu at (147.9, 179.0)
- added R_Pfb2: 68k, Resistor_SMD:R_0603_1608Metric_Pad0.98x0.95mm_HandSolder, F.Cu at (147.9, 184.0)
- added SW1: ~, custom_footprints:SW-TH_SS-12D11G5, F.Cu at (70.0, 172.6)
- added TP21: TestPoint, TestPoint:TestPoint_Pad_D2.0mm, F.Cu at (50.0, 40.0)
- added TP6: TestPoint, TestPoint:TestPoint_Pad_D2.0mm, F.Cu at (66.6, 156.2)
- added TP7: TestPoint, TestPoint:TestPoint_Pad_D2.0mm, F.Cu at (35.6, 163.2)
- added TP8: TestPoint, TestPoint:TestPoint_Pad_D2.0mm, F.Cu at (39.6, 178.2)
- added TP9: TestPoint, TestPoint:TestPoint_Pad_D2.0mm, F.Cu at (34.6, 172.2)
- added TP_3V3: 3V3_OUT, TestPoint:TestPoint_Pad_D2.0mm, F.Cu at (191.0, 160.0)
- added TP_5V0: 5V_OUT, TestPoint:TestPoint_Pad_D2.0mm, F.Cu at (139.0, 177.0)
- added TP_B1: TestPoint, TestPoint:TestPoint_Pad_D2.0mm, F.Cu at (277.0, 67.0)
- added TP_B_Drain3: TestPoint, TestPoint:TestPoint_Pad_D2.0mm, F.Cu at (279.0, 53.0)
- added TP_B_Gate1: TestPoint, TestPoint:TestPoint_Pad_D2.0mm, F.Cu at (278.0, 60.0)
- added TP_B_prog1: charge_prog, TestPoint:TestPoint_Pad_D2.0mm, F.Cu at (268.0, 60.0)
- added TP_B_prog2: charge_gnd, TestPoint:TestPoint_Pad_D2.0mm, F.Cu at (268.0, 53.0)
- added TP_B_sense1: TestPoint, TestPoint:TestPoint_Pad_D2.0mm, F.Cu at (279.6, 155.0)
- added TP_GND0: GND_REF, TestPoint:TestPoint_Pad_D2.0mm, F.Cu at (184.0, 160.0)
- added TP_L1: TestPoint, TestPoint:TestPoint_Pad_D2.0mm, F.Cu at (31.0, 42.0)
- added TP_L2: TestPoint, TestPoint:TestPoint_Pad_D2.0mm, F.Cu at (40.0, 40.0)
- added TP_MA2: TestPoint, TestPoint:TestPoint_Pad_D2.0mm, F.Cu at (184.0, 38.2)
- added TP_MB2: TestPoint, TestPoint:TestPoint_Pad_D2.0mm, F.Cu at (184.0, 30.2)
- added TP_PA1: Boost_ind, TestPoint:TestPoint_Pad_D2.0mm, F.Cu at (132.0, 157.0)
- added TP_PA2: Boost_ind, TestPoint:TestPoint_Pad_D2.0mm, F.Cu at (132.0, 163.0)
- added TP_PB1: Feedback1, TestPoint:TestPoint_Pad_D2.0mm, F.Cu at (132.0, 170.0)
- added TP_PB2: GND, TestPoint:TestPoint_Pad_D2.0mm, F.Cu at (132.0, 177.0)
- added U14: DRV8837DSGR, custom_footprints:SON50P200X200X80-9N, F.Cu at (192.0, 26.9)
- added U15: DRV8837DSGR, custom_footprints:SON50P200X200X80-9N, F.Cu at (192.0, 30.4)
- added U16: DRV8837DSGR, custom_footprints:SON50P200X200X80-9N, F.Cu at (192.0, 34.0)
- added U17: DRV8837DSGR, custom_footprints:SON50P200X200X80-9N, F.Cu at (192.0, 37.5)
- added U2: INA219AxDCN, Package_TO_SOT_SMD:SOT-23-8, F.Cu at (30.0, 99.0)
- added U4: ~, custom_footprints:USB-C-SMD_G-SWITCH_GT-USB-7010ASV, F.Cu at (50.6, 180.2)
- added U5: TPS5430DDA, Package_SO:SOIC-8-1EP_3.9x4.9mm_P1.27mm_EP2.29x3mm, F.Cu at (271.0, 155.0)
- added U6: TP4056-42-ESOP8, custom_footprints:SOIC127P600X175-9N, F.Cu at (270.0, 92.0)
- added U7: AP22966DC8-7, custom_footprints:IC_AP22966DC8-7, F.Cu at (26.0, 22.0)
- added U9: CH224K, Package_SO:SSOP-10-1EP_3.9x4.9mm_P1mm_EP2.1x3.3mm, F.Cu at (50.6, 168.2)
- added U_P1: TPS61022, Package_DFN_QFN:Texas_RWU0007A_VQFN-7_2x2mm_P0.5mm, F.Cu at (138.0, 168.0)
- added U_P2: AMS1117-3.3, Package_TO_SOT_SMD:SOT-223-3_TabPin2, F.Cu at (179.0, 151.0)
Other:
- board outline added: 6.4 x 0.6 mm
