File: Power Board/EEE3088F Power Board/NEW_KICAD/Power_Board_3088F.kicad_pcb (KiCad board)
At the start: 2 copper layers, 6.4 x 0.6 mm, 102 parts, among them J1 Conn_02x16_Odd_Even, J3 Conn_01x02_Socket, Q2 2N7002, U14 DRV8837DSGR, U15 DRV8837DSGR, U16 DRV8837DSGR, U17 DRV8837DSGR, U2 INA219AxDCN, U5 TPS5430DDA, U6 TP4056-42-ESOP8, U7 AP22966DC8-7, U9 CH224K

Commit message: arranged rats nest Tam
Parts:
- moved SW1 96.2 mm to (138.0, 104.6)
- moved U14 89.7 mm to (103.0, 38.0)
- moved TP_MB2 88.9 mm to (96.0, 43.0)
- moved TP_B_sense1 83.4 mm to (231.5, 86.9), turned to -90 degrees
- moved TP_MA2 82.2 mm to (102.0, 43.0)
- moved U16 82.1 mm to (110.0, 38.0)
- moved TP_B1 75.7 mm to (202.0, 77.0)
- moved C_Bin2 74.8 mm to (239.5, 97.9), turned to 90 degrees
- moved TP_B_Gate1 73.1 mm to (208.0, 81.0), turned to 180 degrees
- moved JP_B2 71.5 mm to (224.5, 94.9), turned to -90 degrees
- moved U5 70.6 mm to (234.8, 94.4), turned to -90 degrees
- moved R_Bset3 70.3 mm to (229.5, 94.8), turned to 90 degrees
- moved R_Bset4 68.3 mm to (229.5, 91.9), turned to 180 degrees
- moved TP_B_Drain3 66.7 mm to (218.0, 80.0), turned to 180 degrees
- moved C_B4 64.8 mm to (227.5, 101.9), turned to 90 degrees
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- renumbered D8 to D_CHRG, D4 to D_STBY, TP6 to TP9V, TP8 to TPG8, TP7 to TPVDD
Other:
- board text added: "9V USB C done"
- board text added: "9V buck done"
- board text added: "Charge circuit done"
- board text added: "Git push: Tam: thurs 9:50am"

Commit message: Glen finished organising PCB & some 3D
Parts:
- moved C_P(in)1 53.9 mm to (146.8, 171.2), turned to -90 degrees
- moved JP_P4 48.3 mm to (146.0, 176.2), turned to 180 degrees
- moved C_P(in)3 43.4 mm to (112.6, 166.0)
- moved JP_P3 40.4 mm to (105.3, 164.5)
- moved C_P(in)2 39.7 mm to (153.8, 167.2)
- moved R_P2 39.4 mm to (160.5, 172.2), turned to 90 degrees
- moved 3V3 39.1 mm to (160.2, 168.2), turned to -90 degrees
- moved TP_GND0 38.9 mm to (161.5, 191.7)
- moved 5V0 38.8 mm to (117.1, 178.0)
- moved C_P(out)2 38.5 mm to (125.5, 175.1), turned to -90 degrees
- moved L3 36.5 mm to (105.5, 170.5), turned to -90 degrees
- moved R_Pfb1 35.8 mm to (112.5, 174.0)
- moved R_P1 34.5 mm to (121.0, 178.0), turned to 180 degrees
- moved TP_PA1 34.5 mm to (99.0, 167.0)
- moved TP_3V3 34.4 mm to (160.5, 176.0)
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Other:
- board size 6.4 x 0.6 mm -> 236.6 x 172.9 mm
- board text added: "Battery con Done"
- board text added: "Boost Done"
- board text added: "Current Sensor Done"
- board text added: "Git push: Tam: thurs 9:50am Glen: 12:26"
- board text added: "Ground Test Point for full circ"
- board text added: "LDO Done"
- board text added: "Load Switching Done"
- board text removed: "Git push: Tam: thurs 9:50am"

Commit message: traces started
Parts:
- added H1: MountingHole, MountingHole:MountingHole_3.2mm_M3, F.Cu at (120.0, 76.3)
- moved VDD1 131.3 mm to (144.7, 99.4)
- moved R_C1 130.7 mm to (146.9, 90.7)
- moved R_C2 130.7 mm to (146.9, 94.8)
- moved Bin1 125.6 mm to (114.3, 99.8), turned to -90 degrees
- moved LB1 124.1 mm to (110.9, 91.6), turned to 180 degrees
- moved D7 123.5 mm to (120.2, 101.7), turned to 0 degrees
- moved C_B1 123.4 mm to (116.3, 91.7)
- moved U4 121.3 mm to (136.9, 98.4)
- moved C_C1 119.3 mm to (131.4, 91.8)
- moved R_C3 119.3 mm to (133.4, 85.8)
- moved U9 119.3 mm to (135.4, 90.8)
- moved Vbus_9 119.2 mm to (129.9, 97.3), turned to 90 degrees
- moved TP_5V0 118.2 mm to (92.9, 61.5)
- moved CFG1 117.9 mm to (142.9, 87.4)
- moved GND1 117.8 mm to (143.0, 92.2)
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- renumbered TP9V to 9V1, Batt+1 to B+1, Batt-1 to B-1, TP_B_sense1 to BS1, TP_B_Drain3 to B_D3, TP_B_Gate1 to B_G1, TP_B_prog1 to B_prog1, TP_B_prog2 to B_prog2, JP_B1 to Bin1, TP9 to CFG1, C_Bin2 to C_B1, C_Bboot2 to C_B2, C_C_dd1 to C_C1, C15 to C_L1, C25 to C_L2, C16 to C_L3, C17 to C_L4, C_P(in)3 to C_P1, C_P(out)1 to C_P2, C_P(out)2 to C_P3, C_P(out)3 to C_P4, C_P(in)1 to C_P5, C_P(in)2 to C_P6, D_STBY to D4, D_CHRG to D8, TP_GND0 to GND0, TPG8 to GND1, JP_I1 to J_I1, JP_I2 to J_I2, JPI_3 to J_I3, JP_L2 to J_L2, JP_L1 to J_L3, JP_L3 to L3, L2 to LB1, L3 to L_P3, TP_MA2 to MA2, TP_MB2 to MB2, JP_M_3V3 to M_3V3, JP_M_VM1 to M_VM1, JP_P1 to P1, JP_P2 to P2, JP_P3 to P3, JP_P4 to P4, TP_PA1 to PA1, TP_PA2 to PA2, TP_PB1 to PB1, TP_PB2 to PB2, R_Bset3 to R_B1, R_Bset4 to R_B2, R_B_LED3 to R_B3, R_B_LED4 to R_B4, R_B_b2 to R_B6, R_B_pd2 to R_B7, R_B_fast2 to R_Bfast1, R_B_slow2 to R_Bslow2, R_C_bus1 to R_C1, R_C_dd1 to R_C2, R_C_cfg1 to R_C3, R_Ishunt1 to R_SH1, TP_3V3 to T_3V3, TP_L1 to T_L1, TP_L2 to T_L2, TPVDD to VDD1, JP_CVbus1 to Vbus_9
Connections:
- J_L3 pad 1: Net-(JP_L1-A) -> Net-(J_L3-A)
- U7 pad 4: Net-(JP_L1-A) -> Net-(J_L3-A)
Routing:
- net +9V: track 0.00 -> 143.9 mm
- net /Battery: track 0.00 -> 94.4 mm
- net Net-(U9-VDD): track 0.00 -> 39.3 mm
- net GND: track 0.00 -> 35.7 mm, vias 0 -> 5
- net Net-(Vbus_9-B): track 0.00 -> 25.6 mm
- net Net-(JP_B2-B): track 0.00 -> 22.8 mm
- net /CC1: track 0.00 -> 17.7 mm, vias 0 -> 2
- net Net-(U5-PH): track 0.00 -> 17.4 mm
- net Net-(Q2-G): track 0.00 -> 16.9 mm
- net Net-(U9-VBUS): track 0.00 -> 14.4 mm, vias 0 -> 2
- net Net-(JP_Bprog1-A): track 0.00 -> 14.2 mm
- net Net-(D4-A): track 0.00 -> 14.0 mm
- net Net-(U9-CFG1): track 0.00 -> 11.7 mm
- net Net-(Q2-D): track 0.00 -> 8.69 mm
- net /CC2: track 0.00 -> 8.44 mm
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- added copper zone on B.Cu, net GND
Other:
- board size 236.6 x 172.9 mm -> 60 x 80 mm
- board text added: "Git push: Tam: thurs 9:50am Glen: 12:26 Tam: thurs 18:10pm"
- board text removed: "9V USB C done"
- board text removed: "9V buck done"
- board text removed: "Battery con Done"
- board text removed: "Boost Done"
- board text removed: "Charge circuit done"
- board text removed: "Current Sensor Done"
- board text removed: "Git push: Tam: thurs 9:50am Glen: 12:26"
- board text removed: "Ground Test Point for full circ"
- board text removed: "LDO Done"
- board text removed: "Load Switching Done"

Commit message: Mostly finished Schem
Parts:
- moved PA2 14.9 mm to (97.0, 43.5)
- moved PA1 12.0 mm to (103.0, 43.5)
- moved GND0 9.12 mm to (118.0, 97.0)
- moved B+1 7.82 mm to (94.0, 62.0)
- moved MA2 7.28 mm to (100.0, 36.0)
- moved B-1 7.21 mm to (99.5, 66.0)
- moved R_P2 5.84 mm to (105.1, 76.5), turned to 0 degrees
- moved T_3V3 5.63 mm to (101.5, 77.0)
- moved TP_5V0 5.57 mm to (98.5, 61.5)
- moved MB2 5.52 mm to (95.5, 37.5)
- moved 3V3 5.00 mm to (108.5, 76.5), turned to 180 degrees
- moved J_I1 4.30 mm to (96.0, 78.5), turned to 0 degrees
- moved C_P4 4.26 mm to (115.5, 59.0)
- moved R_I2 4.20 mm to (98.0, 82.0), turned to 0 degrees
- moved PB1 3.70 mm to (102.0, 61.4)
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Routing:
- net +5V: track 0.00 -> 131.7 mm, vias 0 -> 5
- net +BATT: track 3.07 -> 104.3 mm, vias 0 -> 2
- net +3.3V: track 0.00 -> 92.8 mm, vias 0 -> 4
- net /I2C1_SDA: track 0.00 -> 78.5 mm, vias 0 -> 1
- net /I2C1_SCL: track 0.00 -> 70.3 mm, vias 0 -> 1
- net /Switch-: track 0.00 -> 55.3 mm
- net /EXT_LOAD2_OUT: track 0.00 -> 37.6 mm
- net /CTRL_EXT_LOAD1: track 0.00 -> 22.1 mm, vias 0 -> 1
- net Net-(U_P1-SW): track 0.00 -> 21.2 mm, vias 0 -> 2
- net Net-(P1-A): track 0.00 -> 18.5 mm
- net GND: track 35.7 -> 53.9 mm, vias 5 -> 44
- net <NO NET>: track 0.00 -> 18.0 mm, vias 0 -> 2
- net /EXT_LOAD1_OUT: track 0.00 -> 17.7 mm
- net Net-(U_P1-FB): track 0.00 -> 10.3 mm, vias 0 -> 1
- net Net-(L3-A): track 0.00 -> 8.29 mm
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- added copper zone on F.Cu, net +3.3V
- added copper zone on F.Cu, net GND
Other:
- board text added: "Git push: Tam: thurs 9:50am Glen: 12:26 Tam: thurs 18:10pm Glen: Thurs 21:39"
- board text added: "NO HOLES ON SILKSCREENS"
- board text removed: "Git push: Tam: thurs 9:50am Glen: 12:26 Tam: thurs 18:10pm"

Commit message: final v0
Parts:
- D7: footprint custom_footprints:SMA-DIODE -> custom_footprints:B340A
- moved U16 13.0 mm to (105.4, 36.8)
- moved MA2 6.86 mm to (95.0, 31.3)
- moved U14 5.28 mm to (98.4, 36.8)
- moved MB2 4.48 mm to (99.4, 39.7)
- moved P2 1.63 mm to (108.0, 51.8)
- moved R_I1 1.10 mm to (95.0, 85.4)
- moved P1 1.06 mm to (110.8, 53.7)
- moved D7 0.54 mm to (120.3, 100.7), turned to 180 degrees
Connections:
- C_B2 pad 2: Net-(U5-PH) -> Net-(D7-K)
- LB1 pad 1: Net-(U5-PH) -> Net-(D7-K)
- U5 pad 8: Net-(U5-PH) -> Net-(D7-K)
Routing:
- net /FAST_CHARGE_CTRL: track 4.26 -> 95.9 mm, vias 0 -> 1
- net /Battery_VM: track 0.00 -> 69.7 mm, vias 0 -> 4
- net /3V3_M: track 0.00 -> 64.4 mm, vias 0 -> 8
- net /CTRL_EXT_LOAD2: track 0.69 -> 40.7 mm, vias 0 -> 3
- net GND: track 53.9 -> 89.1 mm, vias 44 -> 41
- net /I2C1_SCL: track 70.3 -> 103.8 mm
- net Net-(D4-A): track 14.0 -> 45.3 mm, vias 0 -> 2
- net /5V_Buck_Out: track 2.99 -> 31.2 mm, vias 0 -> 2
- net Net-(D7-K): track 0.00 -> 19.3 mm
- net Net-(U5-PH): track 15.9 -> 0.00 mm
- net /MOTOR2_B_OUT: track 0.00 -> 15.9 mm, vias 0 -> 1
- net /MOTOR2_A_OUT: track 0.00 -> 15.1 mm, vias 0 -> 2
- net /MOTOR2_CTRL2: track 0.00 -> 12.1 mm, vias 0 -> 1
- net Net-(P1-A): track 18.5 -> 30.5 mm
- net /MOTOR4_CTRL2: track 0.00 -> 11.1 mm
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Other:
- outline, holes or cut-outs redrawn
- board text added: "Battery Charging"
- board text added: "Boost"
- board text added: "Group 12"
- board text added: "I Sensor"
- board text added: "LDO"
- board text added: "Load"
- board text added: "M1"
- board text added: "M2"
- board text added: "M3"
- board text added: "M4"
- board text added: "ON"
- board text added: "OSLTAM001 JNSGLE007"
- board text removed: "NO HOLES ON SILKSCREENS"
